File: hardware/wallet_dmm.kicad_pcb (KiCad board)
At the start: 2 copper layers, 85.6 x 54 mm, 67 parts, among them J1 USB-C (charge only), J2 PROBES, J3 OLED 0.91in 128x32 I2C, J4 SWD, J5 LiPo 3.7 V, Q1 AO3401A, Q2 2N7002, SW1 BUTTON A, SW2 BUTTON B, SW3 BUTTON C, SW4 RESET, SW5 POWER, U1 STM32L051K8T6, U2 MCP73831T-2ACI/OT, U3 XC6206P302MR (3.0 V)

Commit message: Firmware, simulation and 3D models for rev 3.
Rust/Embassy firmware for the STM32L051, with the measurement maths and UI
in a host-tested crate. The front end is simulated in ngspice and the
release binary runs in Renode. The simulation found that a fault on the
inputs could pull the 3.0 V rail up while the MCU sleeps, so U4 (TL431)
now clamps it; R13/R14 and C13 changed as well. Every part has a 3D model,
with renders in docs/.
Parts:
- added R29: 330k, Resistor_SMD:R_0603_1608Metric, F.Cu at (124.2, 131.0)
- added R30: 1M, Resistor_SMD:R_0603_1608Metric, F.Cu at (122.4, 131.0)
- added U4: TL431AIDBZR, Package_TO_SOT_SMD:SOT-23, F.Cu at (128.6, 131.0)
- C13: value 100nF -> 22nF
- R13: value 10k -> 4.7k
- R14: value 10k -> 5.1k
Routing:
- net +VSW: track 104.5 -> 138.6 mm, vias 2 -> 0
- net +3V0: track 99.3 -> 132.3 mm, vias 5 -> 4
- net /ADC_ELO: track 38.3 -> 19.0 mm
- net /NRST: track 60.8 -> 71.2 mm, vias 2 -> 1
- net +BATT: track 54.9 -> 64.7 mm, vias 2 -> 1
- net /IN_OHM: track 25.6 -> 35.3 mm, vias 0 -> 1
- net GND: track 143.0 -> 151.6 mm, vias 110 -> 103
- net Net-(U4-REF): track 0.00 -> 8.32 mm
- net Net-(D4-RK): track 17.7 -> 10.8 mm, vias 2 -> 0
- net /VBUS_SENSE: track 25.9 -> 21.8 mm
- net /PIEZO_B: track 25.5 -> 29.0 mm, vias 0 -> 2
- net /E_LO: track 15.7 -> 19.1 mm
- net /OHM_LO: track 11.6 -> 14.6 mm, vias 0 -> 2
- net VBUS: track 37.0 -> 40.0 mm
- net Net-(D4-GK): track 9.79 -> 7.12 mm, vias 0 -> 2
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