File: hardware/wallet_dmm.kicad_sch (KiCad schematic)
At the start: 67 parts, among them J1 USB-C (charge only), J2 PROBES, J3 OLED 0.91in 128x32 I2C, J4 SWD, J5 LiPo 3.7 V, Q1 AO3401A, Q2 2N7002, SW1 BUTTON A, SW2 BUTTON B, SW3 BUTTON C, SW4 RESET, SW5 POWER, U1 STM32L051K8T6, U2 MCP73831T-2ACI/OT, U3 XC6206P302MR (3.0 V)

Commit message: Firmware, simulation and 3D models for rev 3.
Rust/Embassy firmware for the STM32L051, with the measurement maths and UI
in a host-tested crate. The front end is simulated in ngspice and the
release binary runs in Renode. The simulation found that a fault on the
inputs could pull the 3.0 V rail up while the MCU sleeps, so U4 (TL431)
now clamps it; R13/R14 and C13 changed as well. Every part has a 3D model,
with renders in docs/.
Parts:
- added R29: 330k, Resistor_SMD:R_0603_1608Metric, symbol Device:R
- added R30: 1M, Resistor_SMD:R_0603_1608Metric, symbol Device:R
- added U4: TL431AIDBZR, Package_TO_SOT_SMD:SOT-23, symbol Reference_Voltage:TL431DBZ
- C13: value 100nF -> 22nF; LCSC C14663 -> C21122; MPN CC0603KRX7R9BB104 -> CL10B223KB8NNNC; Manufacturer YAGEO -> Samsung Electro-Mechanics
- R13: value 10k -> 4.7k; LCSC C25804 -> C23162; MPN 0603WAF1002T5E -> 0603WAF4701T5E
- R14: value 10k -> 5.1k; LCSC C25804 -> C23186; MPN 0603WAF1002T5E -> 0603WAF5101T5E
Connections:
- net +3V0: now also R29.1, U4.1 (K)
- net GND: now also R30.2, U4.3 (A)
- new net: R29.2, R30.1, U4.2 (REF)
Other:
- note added: "ADC_V = VMID + (VIN - VMID) x R12 / (R10 + R11 + R12) VIN = ADC_V + (ADC_V - VMID) x 20.0; VMID is measured on ADC_VMID. VMID_EN high only while measuring: VMID = 1.56 V, range -31 to +32 V. Overload current is set by R10 + R11 (3 uA at 30 V) into the PA4 clamp."
- note added: "Low range (0-100k, continuity, diode): drive OHM_LO high, RX = R17 x ADC_OHM / (ADC_ELO - ADC_OHM). High range (100k-10M): drive OHM_HI high, RX = R20 x ADC_OHM / (VDD - ADC_OHM). The unused drive pin stays analog (high-Z). Firmware first pulls OHM_LO low: a passive load then reads ~0 V, a source does not. D2/D3 clamp E_LO/E_HI to GND and the battery: 30 V on the input pushes 2.5 mA into the cell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"
- note added: "U4 clamps +3V0 at 3.3 V (2.495 V x (1 + R29 / R30))"
- note removed: "ADC_V = VMID + (VIN - VMID) x R12 / (R10 + R11 + R12) VIN = ADC_V + (ADC_V - VMID) x 20.0; VMID is measured on ADC_VMID. VMID_EN high only while measuring: VMID = 1.5 V, range about +/-31 V. Overload current is set by R10 + R11 (3 uA at 30 V) into the PA4 clamp."
- note removed: "Low range (0-100k, continuity, diode): drive OHM_LO high, RX = R17 x ADC_OHM / (ADC_ELO - ADC_OHM). High range (100k-10M): drive OHM_HI high, RX = R20 x ADC_OHM / (VDD - ADC_OHM). The unused drive pin stays analog (high-Z). D2/D3 clamp E_LO/E_HI to GND and the battery, so 30 V on the input pushes 2.5 mA through R17 into the cell, never into the 3.0 V rail."
